File: labs/schemes/registers/bus.kicad_sch (KiCad schematic)
At the start: 1 part, among them K4 4PDT

Commit message: Some structure updates
Parts:
- K4: footprint (none) -> relay:MY4N socket
Connections:
- net GND: now also K4.13; no longer K4.14
- net SELECT: now also K4.14; no longer K4.13
Changed lines of the file:
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@@
 			)
 		)
-		(property "Footprint" ""
+		(property "Footprint" "relay:MY4N socket"
 			(at 19.05 16.51 0)
 			(effects
