File: labs/schemes/registers/registers.kicad_sch (KiCad schematic)
At the start: 0 parts

Commit message: Many fixes
Other:
- added sheet trigger3 (trigger3.kicad_sch)
Changed lines of the file:
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@@
+	)
+	(sheet
+		(at 133.35 20.32)
+		(size 27.94 22.86)
+		(exclude_from_sim no)
+		(in_bom yes)
+		(on_board yes)
+		(dnp no)
+		(fields_autoplaced yes)
+		(stroke
+			(width 0.1524)
+			(type solid)
+		)
+		(fill
+			(color 0 0 0 0.0000)
+		)
+		(property "Sheetname" "trigger3"
+			(at 133.35 19.6084 0)
+			(effects
+				(font
+					(size 1.27 1.27)
+				)
+				(justify left bottom)
+			)
+		)
+		(property "Sheetfile" "trigger3.kicad_sch"
+			(at 133.35 43.7646 0)
+			(effects
+				(font
+					(size 1.27 1.27)
+				)
+				(justify left top)
+			)
+		)
+		(instances
+			(project "registers"
+				(path "/ab0429f0-9972-454a-bd89-4e26a015f7d3"
+					(page "5")
+				)
+			)
+		)
 	)
 	(sheet
