File: labs/schemes/registers/trigger1.kicad_sch (KiCad schematic)
At the start: 1 part, among them K1 4PDT

Commit message: Some structure updates
Parts:
- K1: footprint (none) -> relay:MY4N socket
Connections:
- net GND: now also K1.13; no longer K1.14
- net SET: now also K1.14; no longer K1.13
Changed lines of the file:
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@@
 			)
 		)
-		(property "Footprint" ""
+		(property "Footprint" "relay:MY4N socket"
 			(at 17.78 11.43 0)
 			(effects

Commit message: Many fixes
Parts:
- added K5, K6: 4PDT, relay:MY4N socket, symbol relay:4PDT
Connections:
- net +: now also K5.12, K6.12
- net GND: now also K5.13, K6.13
- net SET: now also K5.14, K5.8, K6.14, K6.8
