File: labs/schemes/registers/trigger2.kicad_sch (KiCad schematic)
At the start: 2 parts, among them K2 4PDT, K3 4PDT

Commit message: Some structure updates
Parts:
- K2, K3: footprint (none) -> relay:MY4N socket
Connections:
- net GND: now also K2.13, K3.13; no longer K2.14, K3.14
- net RESET: now also K3.14; no longer K3.13
- net SET: now also K2.14; no longer K2.13
Changed lines of the file:
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@@
 			)
 		)
-		(property "Footprint" ""
+		(property "Footprint" "relay:MY4N socket"
 			(at 13.97 10.16 0)
 			(effects
@@
 			)
 		)
-		(property "Footprint" ""
+		(property "Footprint" "relay:MY4N socket"
 			(at 50.8 10.16 0)
 			(effects
