File: labs/schemes/operations/operations.kicad_sch (KiCad schematic)
At the start: 0 parts

Commit message: Many updates
Other:
- added sheet add (add.kicad_sch)
- added sheet not (not.kicad_sch)
- added sheet shr (shr.kicad_sch)
Changed lines of the file:
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@@
+	)
+	(sheet
+		(at 86.36 46.99)
+		(size 20.32 16.51)
+		(exclude_from_sim no)
+		(in_bom yes)
+		(on_board yes)
+		(dnp no)
+		(fields_autoplaced yes)
+		(stroke
+			(width 0.1524)
+			(type solid)
+		)
+		(fill
+			(color 0 0 0 0.0000)
+		)
+		(property "Sheetname" "add"
+			(at 86.36 46.2784 0)
+			(effects
+				(font
+					(size 1.27 1.27)
+				)
+				(justify left bottom)
+			)
+		)
+		(property "Sheetfile" "add.kicad_sch"
+			(at 86.36 64.0846 0)
+			(effects
+				(font
+					(size 1.27 1.27)
+				)
+				(justify left top)
+			)
+		)
+		(instances
+			(project "operations"
+				(path "/ef21cd22-a9e7-4e45-b09f-de717f45c340"
+					(page "8")
+				)
+			)
+		)
 	)
 	(sheet
@@
 	)
 	(sheet
+		(at 25.4 46.99)
+		(size 22.86 16.51)
+		(exclude_from_sim no)
+		(in_bom yes)
+		(on_board yes)
+		(dnp no)
+		(fields_autoplaced yes)
+		(stroke
+			(width 0.1524)
+			(type solid)
+		)
+		(fill
+			(color 0 0 0 0.0000)
+		)
+		(property "Sheetname" "not"
+			(at 25.4 46.2784 0)
+			(effects
+				(font
+					(size 1.27 1.27)
+				)
+				(justify left bottom)
+			)
+		)
+		(property "Sheetfile" "not.kicad_sch"
+			(at 25.4 64.0846 0)
+			(effects
+				(font
+					(size 1.27 1.27)
+				)
+				(justify left top)
+			)
+		)
+		(instances
+			(project "operations"
+				(path "/ef21cd22-a9e7-4e45-b09f-de717f45c340"
+					(page "6")
+				)
+			)
+		)
+	)
+	(sheet
 		(at 25.4 21.59)
 		(size 22.86 15.24)
@@
 				)
 			)
+		)
+	)
+	(sheet
+		(at 55.88 46.99)
+		(size 20.32 16.51)
+		(exclude_from_sim no)
+		(in_bom yes)
+		(on_board yes)
+		(dnp no)
+		(fields_autoplaced yes)
+		(stroke
+			(width 0.1524)
+			(type solid)
+		)
+		(fill
+			(color 0 0 0 0.0000)
+		)
+		(property "Sheetname" "shr"
+			(at 55.88 46.2784 0)
+			(effects
+				(font
+					(size 1.27 1.27)
+				)
+				(justify left bottom)
+			)
+		)
+		(property "Sheetfile" "shr.kicad_sch"
+			(at 55.88 64.0846 0)
+			(effects
+				(font
+					(size 1.27 1.27)
+				)
+				(justify left top)
+			)
+		)
+		(instances
+			(project "operations"
+				(path "/ef21cd22-a9e7-4e45-b09f-de717f45c340"
+					(page "7")
+				)
+			)

Commit message: Many updates
Other:
- added sheet switches_and (switches_and.kicad_sch)
- added sheet switches_or (switches_or.kicad_sch)
Changed lines of the file:
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@@
+	)
+	(sheet
+		(at 25.4 91.44)
+		(size 22.86 15.24)
+		(exclude_from_sim no)
+		(in_bom yes)
+		(on_board yes)
+		(dnp no)
+		(fields_autoplaced yes)
+		(stroke
+			(width 0.1524)
+			(type solid)
+		)
+		(fill
+			(color 0 0 0 0.0000)
+		)
+		(property "Sheetname" "switches_and"
+			(at 25.4 90.7284 0)
+			(effects
+				(font
+					(size 1.27 1.27)
+				)
+				(justify left bottom)
+			)
+		)
+		(property "Sheetfile" "switches_and.kicad_sch"
+			(at 25.4 107.2646 0)
+			(effects
+				(font
+					(size 1.27 1.27)
+				)
+				(justify left top)
+			)
+		)
+		(instances
+			(project "operations"
+				(path "/ef21cd22-a9e7-4e45-b09f-de717f45c340"
+					(page "9")
+				)
+			)
+		)
 	)
 	(sheet
@@
 				)
 			)
+		)
+	)
+	(sheet
+		(at 58.42 91.44)
+		(size 22.86 15.24)
+		(exclude_from_sim no)
+		(in_bom yes)
+		(on_board yes)
+		(dnp no)
+		(fields_autoplaced yes)
+		(stroke
+			(width 0.1524)
+			(type solid)
+		)
+		(fill
+			(color 0 0 0 0.0000)
+		)
+		(property "Sheetname" "switches_or"
+			(at 58.42 90.7284 0)
+			(effects
+				(font
+					(size 1.27 1.27)
+				)
+				(justify left bottom)
+			)
+		)
+		(property "Sheetfile" "switches_or.kicad_sch"
+			(at 58.42 107.2646 0)
+			(effects
+				(font
+					(size 1.27 1.27)
+				)
+				(justify left top)
+			)
+		)
+		(instances
+			(project "operations"
+				(path "/ef21cd22-a9e7-4e45-b09f-de717f45c340"
+					(page "10")
+				)
+			)
