File: labs/schemes/operations/add.kicad_sch (KiCad schematic)
At the start: 2 parts, among them K7 4PDT, K8 4PDT

Commit message: Some structure updates
Connections:
- net GND: now also K7.13, K8.13; no longer K7.14, K8.14
- net IN1: now also K7.14; no longer K7.13
- net IN2: now also K8.14; no longer K8.13
