File: labs/schemes/operations/and.kicad_sch (KiCad schematic)
At the start: 1 part, among them K1 4PDT

Commit message: Some structure updates
Parts:
- K1: footprint (none) -> relay:MY4N socket
Connections:
- net B: now also K1.14; no longer K1.13
- net GND: now also K1.13; no longer K1.14
Changed lines of the file:
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@@
 			)
 		)
-		(property "Footprint" ""
+		(property "Footprint" "relay:MY4N socket"
 			(at 19.05 21.59 0)
 			(effects

Commit message: Many updates
Parts:
- K1: symbol relay:4PDT -> relay:SPDT
Connections:
- net A: now also K1.12; no longer K1.9
- net C: now also K1.8; no longer K1.5
Changed lines of the file:
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@@
 	(generator "eeschema")
 	(generator_version "9.0")
-	(paper "User" 46.99 54.61)
-	(wire
-		(pts
-			(xy 35.56 20.32) (xy 40.64 20.32)
+	(paper "A4" portrait)
+	(wire
+		(pts
+			(xy 35.56 35.56) (xy 40.64 35.56)
 		)
 		(stroke
@@
 	(wire
 		(pts
-			(xy 16.51 20.32) (xy 21.59 20.32)
+			(xy 16.51 35.56) (xy 21.59 35.56)
 		)
 		(stroke
@@
 	)
 	(label "C"
-		(at 39.37 20.32 0)
+		(at 39.37 35.56 0)
 		(effects
 			(font
@@
 	)
 	(label "A"
-		(at 16.51 20.32 0)
+		(at 16.51 35.56 0)
 		(effects
 			(font
@@
 	)
 	(symbol
-		(lib_id "relay:4PDT")
+		(lib_id "relay:SPDT")
 		(at 19.05 21.59 0)
 		(unit 1)
@@
 		)
 		(property "Footprint" "relay:MY4N socket"
-			(at 19.05 21.59 0)
+			(at 10.922 80.264 0)
 			(effects
 				(font
@@
 		(pin "8"
 		)
-		(pin "7"
-		)
-		(pin "1"
-		)
-		(pin "9"
-		)
 		(pin "4"
 		)
-		(pin "11"
-		)
-		(pin "10"
-		)
-		(pin "6"
-		)
-		(pin "5"
-		)
-		(pin "3"
-		)
-		(pin "2"
-		)
 		(instances
