File: labs/schemes/operations/not.kicad_sch (KiCad schematic)
At the start: 1 part, among them K6 4PDT

Commit message: Some structure updates
Parts:
- K6: footprint (none) -> relay:MY4N socket
Connections:
- net A: now also K6.14; no longer K6.13
- net GND: now also K6.13; no longer K6.14
Changed lines of the file:
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@@
 			)
 		)
-		(property "Footprint" ""
+		(property "Footprint" "relay:MY4N socket"
 			(at 12.7 11.43 0)
 			(effects

Commit message: Many updates
Parts:
- K6: symbol relay:4PDT -> relay:SPDT
Connections:
- net C: now reaches K6.8
Changed lines of the file:
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@@
+		)
+	)
+	(wire
+		(pts
+			(xy 29.21 25.4) (xy 38.1 25.4)
+		)
+		(stroke
+			(width 0)
+			(type default)
 		)
 	)
@@
 	(label "+"
 		(at 6.35 25.4 0)
+		(effects
+			(font
+				(size 1.27 1.27)
+			)
+			(justify left bottom)
+		)
+	)
+	(label "C"
+		(at 36.83 25.4 0)
 		(effects
 			(font
@@
 	)
 	(symbol
-		(lib_id "relay:4PDT")
+		(lib_id "relay:SPDT")
 		(at 12.7 11.43 0)
 		(unit 1)
@@
 		)
 		(property "Value" "4PDT"
-			(at 22.225 3.81 0)
+			(at 22.352 19.558 0)
 			(effects
 				(font
@@
 		)
 		(property "Footprint" "relay:MY4N socket"
-			(at 12.7 11.43 0)
+			(at 4.572 70.104 0)
 			(effects
 				(font
@@
 		(pin "12"
 		)
-		(pin "5"
-		)
-		(pin "1"
-		)
 		(pin "13"
-		)
-		(pin "11"
-		)
-		(pin "10"
-		)
-		(pin "9"
-		)
-		(pin "2"
-		)
-		(pin "7"
 		)
 		(pin "14"
@@
 		(pin "8"
 		)
-		(pin "3"
-		)
 		(pin "4"
 		)
-		(pin "6"
-		)
 		(instances
