File: labs/schemes/relay/diode.kicad_sch (KiCad schematic)
At the start: 6 parts, among them K2 4PDT, K3 4PDT, SW1 SW_DPST_x2, SW2 SW_DPST_x2

Commit message: Some structure updates
Parts:
- K2, K3: footprint (none) -> relay:MY4N socket
Connections:
- net GND: now also K2.13, K3.13; no longer K2.14, K3.14
- net at D2.1 (K), SW2.2 (B): now also K3.14; no longer K3.13
- net at D1.1 (K), SW1.2 (B): now also K2.14; no longer K2.13
Changed lines of the file:
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@@
 			)
 		)
-		(property "Footprint" ""
+		(property "Footprint" "relay:MY4N socket"
 			(at 69.85 11.43 0)
 			(effects
@@
 			)
 		)
-		(property "Footprint" ""
+		(property "Footprint" "relay:MY4N socket"
 			(at 22.86 11.43 0)
 			(effects
@@
 			)
 		)
+		(property "Sim.Enable" "0"
+			(at 88.9 44.45 0)
+			(effects
+				(font
+					(size 1.27 1.27)
+				)
+				(hide yes)
+			)
+		)
 		(instances
 			(project "relay"
@@
 		(at 41.91 45.72 270)
 		(unit 1)
-		(exclude_from_sim no)
+		(exclude_from_sim yes)
 		(in_bom no)
 		(on_board no)
