File: labs/schemes/relay/relay.kicad_sch (KiCad schematic)
At the start: 0 parts

Commit message: Many updates
Other:
- added sheet simple_relay_off (simple_relay_off.kicad_sch)
- added sheet simple_relay_on (simple_relay_on.kicad_sch)
Changed lines of the file:
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@@
+	)
+	(sheet
+		(at 110.49 16.51)
+		(size 16.51 16.51)
+		(exclude_from_sim no)
+		(in_bom yes)
+		(on_board yes)
+		(dnp no)
+		(fields_autoplaced yes)
+		(stroke
+			(width 0.1524)
+			(type solid)
+		)
+		(fill
+			(color 0 0 0 0.0000)
+		)
+		(property "Sheetname" "simple_relay_on"
+			(at 110.49 15.7984 0)
+			(effects
+				(font
+					(size 1.27 1.27)
+				)
+				(justify left bottom)
+			)
+		)
+		(property "Sheetfile" "simple_relay_on.kicad_sch"
+			(at 110.49 33.6046 0)
+			(effects
+				(font
+					(size 1.27 1.27)
+				)
+				(justify left top)
+			)
+		)
+		(instances
+			(project "relay"
+				(path "/5c1fc490-b475-4768-befc-b1eff004344c"
+					(page "5")
+				)
+			)
+		)
 	)
 	(sheet
@@
 				)
 			)
+		)
+	)
+	(sheet
+		(at 73.66 16.51)
+		(size 16.51 16.51)
+		(exclude_from_sim no)
+		(in_bom yes)
+		(on_board yes)
+		(dnp no)
+		(fields_autoplaced yes)
+		(stroke
+			(width 0.1524)
+			(type solid)
+		)
+		(fill
+			(color 0 0 0 0.0000)
+		)
+		(property "Sheetname" "simple_relay_off"
+			(at 73.66 15.7984 0)
+			(effects
+				(font
+					(size 1.27 1.27)
+				)
+				(justify left bottom)
+			)
+		)
+		(property "Sheetfile" "simple_relay_off.kicad_sch"
+			(at 73.66 33.6046 0)
+			(effects
+				(font
+					(size 1.27 1.27)
+				)
+				(justify left top)
+			)
+		)
+		(instances
+			(project "relay"
+				(path "/5c1fc490-b475-4768-befc-b1eff004344c"
+					(page "4")
+				)
+			)
