File: labs/schemes/relay/one_relay.kicad_sch (KiCad schematic)
At the start: 1 part, among them K1 4PDT

Commit message: Some structure updates
Parts:
- K1: footprint (none) -> relay:MY4N socket
Changed lines of the file:
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@@
 			)
 		)
-		(property "Footprint" ""
+		(property "Footprint" "relay:MY4N socket"
 			(at 3.81 12.7 0)
 			(effects

Commit message: Many updates
Parts:
- added K6: FRT5_separated, Relay_THT:Relay_DPDT_FRT5, symbol Relay:FRT5_separated
