File: modules/power/power.kicad_pcb (KiCad board)
At the start: 2 copper layers, 49 x 42 mm, 5 parts, among them J1 Jack-DC

Commit message: Added bus module
Other:
- board text added: "Power"
Changed lines of the file:
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@@
+		)
+	)
+	(gr_text "Power"
+		(at 148.5 96.5 0)
+		(layer "Dwgs.User")
+		(effects
+			(font
+				(size 5 5)
+				(thickness 0.625)
+			)
+			(justify left bottom)
 		)
 	)
