File: modules/power/power.kicad_pcb (KiCad board)
At the start: 2 copper layers, 49 x 42 mm, 5 parts, among them J1 Jack-DC

Commit message: Added BOM calculation
Other:
- board text added: "Power board v1.0 P. Dovgalyuk, 2026"
- board text removed: "Power board rev6 P. Dovgalyuk, 2026"
Changed lines of the file:
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@@
 		(layer "Edge.Cuts")
 	)
-	(gr_text "Power board rev6\nP. Dovgalyuk, 2026"
+	(gr_text "Power board v1.0\nP. Dovgalyuk, 2026"
 		(at 172 97.5 0)
 		(layer "B.SilkS")
