File: modules/adder/adder.kicad_pcb (KiCad board)
At the start: 2 copper layers, 120 x 109.5 mm, 26 parts, among them J1 IN1, J10 CY/~CY, J11 CY_OUT, J2 IN2, J3 OUT, J5 IN1, J6 OUT, J7 IN2, K1 4PDT, K2 4PDT, K3 4PDT, K4 4PDT, K5 4PDT, K6 4PDT, K7 4PDT, K8 4PDT

Commit message: Added BOM calculation
Connections:
- net Net-(J1-+V) renamed +24V
Routing:
- net +24V: track 533.7 -> 0.00 mm
- net GND: track 481.8 -> 0.00 mm
- net Net-(D7-K): track 115.0 -> 154.6 mm
- net Net-(D8-K): track 154.7 -> 118.0 mm
- net Net-(D6-K): track 176.5 -> 142.4 mm
- net Net-(D3-K): track 73.1 -> 77.1 mm
- net Net-(K3-Pad11): track 72.8 -> 75.5 mm
- net Net-(J3-D1): track 37.9 -> 40.5 mm
- net Net-(J3-D3): track 53.5 -> 55.4 mm
- net Net-(K5-Pad11): track 72.8 -> 74.7 mm
- net Net-(J10-Pin_3): track 82.8 -> 84.6 mm
- net Net-(D1-K): track 130.4 -> 131.7 mm
- net Net-(K1-Pad11): track 72.0 -> 73.0 mm
- net Net-(J3-D0): track 88.3 -> 87.3 mm
- net Net-(D5-K): track 90.2 -> 90.9 mm
- added copper zone on F.Cu, net +24V
- added copper zone on B.Cu, net GND
Other:
- board text added: "Adder"
- board text added: "Adder board v1.0 P. Dovgalyuk, 2026"
- board text added: "In1"
- board text added: "In2"
- board text added: "Out"
- board text removed: "ADD"
- board text removed: "Adder board rev4 P. Dovgalyuk, 2025"
- board text removed: "IN1"
- board text removed: "IN2"
