File: modules/adder/adder.kicad_sch (KiCad schematic)
At the start: 26 parts, among them J1 IN1, J10 CY/~CY, J11 CY_OUT, J2 IN2, J3 OUT, J5 IN1, J6 OUT, J7 IN2, K1 4PDT, K2 4PDT, K3 4PDT, K4 4PDT, K5 4PDT, K6 4PDT, K7 4PDT, K8 4PDT

Commit message: Added BOM calculation
Connections:
- net +24V: now reaches J1.1 (+V), J10.2 (Pin_2), J11.1 (+V), J2.1 (+V), J3.1 (+V), J5.1 (+V), J6.1 (+V), J7.1 (+V), J8.1 (+V), J9.1 (+V), K2.10, K4.10, K6.10, K8.10
Changed lines of the file:
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@@
 	)
 	(junction
+		(at 36.83 58.42)
+		(diameter 0)
+		(color 0 0 0 0)
+	)
+	(junction
 		(at 260.35 111.76)
 		(diameter 0)
@@
 	(wire
 		(pts
+			(xy 36.83 50.8) (xy 36.83 58.42)
+		)
+		(stroke
+			(width 0)
+			(type default)
+		)
+	)
+	(wire
+		(pts
 			(xy 265.43 144.78) (xy 265.43 119.38)
 		)
@@
 		)
 		(instances
-			(project ""
+			(project "adder"
 				(path "/00847eda-8256-4c41-8936-f4fb88f58f68"
 					(reference "K3")
@@
 		)
 		(instances
-			(project ""
+			(project "adder"
 				(path "/00847eda-8256-4c41-8936-f4fb88f58f68"
 					(reference "K7")
@@
 		)
 		(instances
-			(project ""
+			(project "adder"
 				(path "/00847eda-8256-4c41-8936-f4fb88f58f68"
 					(reference "J9")
@@
 		)
 		(instances
-			(project ""
+			(project "adder"
 				(path "/00847eda-8256-4c41-8936-f4fb88f58f68"
 					(reference "D6")
@@
 		)
 		(instances
-			(project ""
+			(project "adder"
 				(path "/00847eda-8256-4c41-8936-f4fb88f58f68"
 					(reference "D8")
@@
 	)
 	(symbol
+		(lib_id "power:+24V")
+		(at 36.83 50.8 0)
+		(unit 1)
+		(exclude_from_sim no)
+		(in_bom yes)
+		(on_board yes)
+		(dnp no)
+		(fields_autoplaced yes)
+		(property "Reference" "#PWR02"
+			(at 36.83 54.61 0)
+			(effects
+				(font
+					(size 1.27 1.27)
+				)
+				(hide yes)
+			)
+		)
+		(property "Value" "+24V"
+			(at 36.83 45.72 0)
+			(effects
+				(font
+					(size 1.27 1.27)
+				)
+			)
+		)
+		(property "Footprint" ""
+			(at 36.83 50.8 0)
+			(effects
+				(font
+					(size 1.27 1.27)
+				)
+				(hide yes)
+			)
+		)
+		(property "Datasheet" ""
+			(at 36.83 50.8 0)
+			(effects
+				(font
+					(size 1.27 1.27)
+				)
+				(hide yes)
+			)
+		)
+		(property "Description" "Power symbol creates a global label with name \"+24V\""
+			(at 36.83 50.8 0)
+			(effects
+				(font
+					(size 1.27 1.27)
+				)
+				(hide yes)
+			)
+		)
+		(pin "1"
+		)
+		(instances
+			(project "adder"
+				(path "/00847eda-8256-4c41-8936-f4fb88f58f68"
+					(reference "#PWR02")
+					(unit 1)
+				)
+			)
+		)
+	)
+	(symbol
 		(lib_id "relay:4PDT")
 		(at 171.45 77.47 0)
@@
 		)
 		(instances
-			(project ""
+			(project "adder"
 				(path "/00847eda-8256-4c41-8936-f4fb88f58f68"
 					(reference "K6")
@@
 		)
 		(instances
-			(project ""
+			(project "adder"
 				(path "/00847eda-8256-4c41-8936-f4fb88f58f68"
 					(reference "K1")
@@
 		)
 		(instances
-			(project ""
+			(project "adder"
 				(path "/00847eda-8256-4c41-8936-f4fb88f58f68"
 					(reference "D3")
@@
 		)
 		(instances
-			(project ""
+			(project "adder"
 				(path "/00847eda-8256-4c41-8936-f4fb88f58f68"
 					(reference "D4")
@@
 		)
 		(instances
-			(project ""
+			(project "adder"
 				(path "/00847eda-8256-4c41-8936-f4fb88f58f68"
 					(reference "K2")
@@
 		)
 		(instances
-			(project ""
+			(project "adder"
 				(path "/00847eda-8256-4c41-8936-f4fb88f58f68"
 					(reference "D7")
@@
 		)
 		(instances
-			(project ""
+			(project "adder"
 				(path "/00847eda-8256-4c41-8936-f4fb88f58f68"
 					(reference "D2")
@@
 		)
 		(instances
-			(project ""
+			(project "adder"
 				(path "/00847eda-8256-4c41-8936-f4fb88f58f68"
 					(reference "K5")
@@
 		)
 		(instances
-			(project ""
+			(project "adder"
 				(path "/00847eda-8256-4c41-8936-f4fb88f58f68"
 					(reference "D5")
@@
 		)
 		(instances
-			(project ""
+			(project "adder"
 				(path "/00847eda-8256-4c41-8936-f4fb88f58f68"
 					(reference "D1")
@@
 		)
 		(instances
-			(project ""
+			(project "adder"
 				(path "/00847eda-8256-4c41-8936-f4fb88f58f68"
 					(reference "J2")
@@
 		)
 		(instances
-			(project ""
+			(project "adder"
 				(path "/00847eda-8256-4c41-8936-f4fb88f58f68"
 					(reference "#PWR01")
@@
 		)
 		(instances
-			(project ""
+			(project "adder"
 				(path "/00847eda-8256-4c41-8936-f4fb88f58f68"
 					(reference "J3")
@@
 		)
 		(instances
-			(project ""
+			(project "adder"
 				(path "/00847eda-8256-4c41-8936-f4fb88f58f68"
 					(reference "J8")
@@
 		)
 		(instances
-			(project ""
+			(project "adder"
 				(path "/00847eda-8256-4c41-8936-f4fb88f58f68"
 					(reference "J10")
@@
 		)
 		(instances
-			(project ""
+			(project "adder"
 				(path "/00847eda-8256-4c41-8936-f4fb88f58f68"
 					(reference "K8")
@@
 		)
 		(instances
-			(project ""
+			(project "adder"
 				(path "/00847eda-8256-4c41-8936-f4fb88f58f68"
 					(reference "K4")
@@
 		)
 		(instances
-			(project ""
+			(project "adder"
 				(path "/00847eda-8256-4c41-8936-f4fb88f58f68"
 					(reference "J1")
