File: modules/binary/binary.kicad_pcb (KiCad board)
At the start: 2 copper layers, 122 x 114.5 mm, 28 parts, among them J10 AND, J11 OR, J12 XOR, J3 IN1, J4 IN2, J5 AND, J6 OR, J7 XOR, J8 IN1, J9 IN2, K1 4PDT, K2 4PDT, K3 4PDT, K4 4PDT, K5 4PDT, K6 4PDT, K7 4PDT, K8 4PDT

Commit message: Added BOM calculation
Other:
- board text added: "Binary logic board v1.0 P. Dovgalyuk, 2026"
- board text removed: "Binary logic board rev6 P. Dovgalyuk, 2026"
Changed lines of the file:
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@@
 			(drillshape 0)
 			(scaleselection 1)
-			(outputdirectory "../../gerber/rev2/logic_binary")
+			(outputdirectory "../../gerber/rev2/binary")
 		)
 	)
@@
 		)
 		(sheetname "/")
-		(sheetfile "logic_binary.kicad_sch")
+		(sheetfile "binary.kicad_sch")
 		(attr through_hole)
 		(fp_rect
@@
 		)
 		(sheetname "/")
-		(sheetfile "logic_binary.kicad_sch")
+		(sheetfile "binary.kicad_sch")
 		(attr through_hole)
 		(fp_rect
@@
 		(property ki_fp_filters "D*DO?35*")
 		(sheetname "/")
-		(sheetfile "logic_binary.kicad_sch")
+		(sheetfile "binary.kicad_sch")
 		(attr through_hole)
 		(fp_line
@@
 		)
 		(sheetname "/")
-		(sheetfile "logic_binary.kicad_sch")
+		(sheetfile "binary.kicad_sch")
 		(attr through_hole)
 		(fp_line
@@
 		)
 		(sheetname "/")
-		(sheetfile "logic_binary.kicad_sch")
+		(sheetfile "binary.kicad_sch")
 		(attr through_hole)
 		(fp_rect
@@
 		)
 		(sheetname "/")
-		(sheetfile "logic_binary.kicad_sch")
+		(sheetfile "binary.kicad_sch")
 		(attr through_hole)
 		(fp_line
@@
 		(property ki_fp_filters "D*DO?35*")
 		(sheetname "/")
-		(sheetfile "logic_binary.kicad_sch")
+		(sheetfile "binary.kicad_sch")
 		(attr through_hole)
 		(fp_line
@@
 		)
 		(sheetname "/")
-		(sheetfile "logic_binary.kicad_sch")
+		(sheetfile "binary.kicad_sch")
 		(attr through_hole)
 		(fp_line
@@
 		)
 		(sheetname "/")
-		(sheetfile "logic_binary.kicad_sch")
+		(sheetfile "binary.kicad_sch")
 		(attr through_hole)
 		(fp_rect
@@
 		)
 		(sheetname "/")
-		(sheetfile "logic_binary.kicad_sch")
+		(sheetfile "binary.kicad_sch")
 		(attr through_hole)
 		(fp_line
@@
 		)
 		(sheetname "/")
-		(sheetfile "logic_binary.kicad_sch")
+		(sheetfile "binary.kicad_sch")
 		(attr through_hole)
 		(fp_rect
@@
 		)
 		(sheetname "/")
-		(sheetfile "logic_binary.kicad_sch")
+		(sheetfile "binary.kicad_sch")
 		(attr through_hole)
 		(fp_line
@@
 		)
 		(sheetname "/")
-		(sheetfile "logic_binary.kicad_sch")
+		(sheetfile "binary.kicad_sch")
 		(attr through_hole)
 		(fp_line
@@
 		(property ki_fp_filters "D*DO?35*")
 		(sheetname "/")
-		(sheetfile "logic_binary.kicad_sch")
+		(sheetfile "binary.kicad_sch")
 		(attr through_hole)
 		(fp_line
@@
 		(property ki_fp_filters "D*DO?35*")
 		(sheetname "/")
-		(sheetfile "logic_binary.kicad_sch")
+		(sheetfile "binary.kicad_sch")
 		(attr through_hole)
 		(fp_line
@@
 		)
 		(sheetname "/")
-		(sheetfile "logic_binary.kicad_sch")
+		(sheetfile "binary.kicad_sch")
 		(attr through_hole)
 		(fp_rect
@@
 		)
 		(sheetname "/")
-		(sheetfile "logic_binary.kicad_sch")
+		(sheetfile "binary.kicad_sch")
 		(attr through_hole)
 		(fp_line
@@
 		(property ki_fp_filters "D*DO?35*")
 		(sheetname "/")
-		(sheetfile "logic_binary.kicad_sch")
+		(sheetfile "binary.kicad_sch")
 		(attr through_hole)
 		(fp_line
@@
 		(property ki_fp_filters "D*DO?35*")
 		(sheetname "/")
-		(sheetfile "logic_binary.kicad_sch")
+		(sheetfile "binary.kicad_sch")
 		(attr through_hole)
 		(fp_line
@@
 		)
 		(sheetname "/")
-		(sheetfile "logic_binary.kicad_sch")
+		(sheetfile "binary.kicad_sch")
 		(attr through_hole)
 		(fp_line
@@
 		)
 		(sheetname "/")
-		(sheetfile "logic_binary.kicad_sch")
+		(sheetfile "binary.kicad_sch")
 		(attr through_hole)
 		(fp_rect
@@
 		)
 		(sheetname "/")
-		(sheetfile "logic_binary.kicad_sch")
+		(sheetfile "binary.kicad_sch")
 		(attr through_hole)
 		(fp_line
@@
 		)
 		(sheetname "/")
-		(sheetfile "logic_binary.kicad_sch")
+		(sheetfile "binary.kicad_sch")
 		(attr through_hole)
 		(fp_line
@@
 		)
 		(sheetname "/")
-		(sheetfile "logic_binary.kicad_sch")
+		(sheetfile "binary.kicad_sch")
 		(attr through_hole)
 		(fp_line
@@
 		)
 		(sheetname "/")
-		(sheetfile "logic_binary.kicad_sch")
+		(sheetfile "binary.kicad_sch")
 		(attr through_hole)
 		(fp_rect
@@
 		)
 		(sheetname "/")
-		(sheetfile "logic_binary.kicad_sch")
+		(sheetfile "binary.kicad_sch")
 		(attr through_hole)
 		(fp_line
@@
 		(property ki_fp_filters "D*DO?35*")
 		(sheetname "/")
-		(sheetfile "logic_binary.kicad_sch")
+		(sheetfile "binary.kicad_sch")
 		(attr through_hole)
 		(fp_line
@@
 		(property ki_fp_filters "D*DO?35*")
 		(sheetname "/")
-		(sheetfile "logic_binary.kicad_sch")
+		(sheetfile "binary.kicad_sch")
 		(attr through_hole)
 		(fp_line
@@
 		(layer "Edge.Cuts")
 	)
-	(gr_text "Or"
-		(at 138.5 128.425855 0)
-		(layer "F.SilkS")
-		(effects
-			(font
-				(size 4 4)
-				(thickness 0.5)
-			)
-			(justify left bottom)
-		)
-	)
 	(gr_text "And"
 		(at 93.5 137.425855 0)
@@
 		)
 	)
-	(gr_text "Binary"
-		(at 88.61 66.425855 90)
+	(gr_text "Or"
+		(at 138.5 128.425855 0)
 		(layer "F.SilkS")
 		(effects
 			(font
-				(size 5 5)
-				(thickness 0.625)
+				(size 4 4)
+				(thickness 0.5)
 			)
 			(justify left bottom)
@@
 		)
 	)
-	(gr_text "Binary logic board rev6\nP. Dovgalyuk, 2026"
+	(gr_text "Binary"
+		(at 88.61 66.425855 90)
+		(layer "F.SilkS")
+		(effects
+			(font
+				(size 5 5)
+				(thickness 0.625)
+			)
+			(justify left bottom)
+		)
+	)
+	(gr_text "Binary logic board v1.0\nP. Dovgalyuk, 2026"
 		(at 199.5 150.925855 0)
 		(layer "B.SilkS")
@@
 		)
 	)
-	(gr_text "Результат\nИСКЛЮЧАЮЩЕЕ ИЛИ"
-		(at 153.5 163 0)
+	(gr_text "Операнд 1"
+		(at 93 28.5 0)
 		(layer "Dwgs.User")
 		(effects
@@
 		)
 	)
-	(gr_text "Питание"
-		(at 213 98 90)
+	(gr_text "Результат\nИ"
+		(at 104.5 163 0)
 		(layer "Dwgs.User")
 		(effects
@@
 		)
 	)
-	(gr_text "Операнд 1"
-		(at 93 28.5 0)
+	(gr_text "Результат\nИСКЛЮЧАЮЩЕЕ ИЛИ"
+		(at 153.5 163 0)
 		(layer "Dwgs.User")
 		(effects
@@
 		)
 	)
-	(gr_text "Результат\nИ"
-		(at 104.5 163 0)
+	(gr_text "Питание"
+		(at 213 98 90)
 		(layer "Dwgs.User")
 		(effects
