File: modules/bus/bus.kicad_pcb (KiCad board)
At the start: 2 copper layers, 84.5 x 25.8 mm, 6 parts

Commit message: Added BOM calculation
Other:
- board text added: "Bus board v1.0 P. Dovgalyuk, 2026"
- board text removed: "Bus board rev6 P. Dovgalyuk, 2026"
Changed lines of the file:
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@@
 		)
 	)
-	(gr_text "Bus board rev6\nP. Dovgalyuk, 2026"
+	(gr_text "Bus board v1.0\nP. Dovgalyuk, 2026"
 		(at 161.5 99 0)
 		(layer "B.SilkS")
