File: modules/clock/clock.kicad_pcb (KiCad board)
At the start: 2 copper layers, 100 x 85 mm, 20 parts, among them J1 OUT, J3 RIGHT, J4 RIGHT, J5 LEFT, J6 LEFT, J7 OUT, K1 4PDT, K2 4PDT, K3 4PDT, K4 4PDT, SW1 On/Off, SW3 Start

Commit message: Updated actions
Parts:
- added D5: 1N4148, Diode_THT:D_DO-35_SOD27_P7.62mm_Horizontal, F.Cu at (120.7, 114.2)
- added D6: 1N4148, Diode_THT:D_DO-35_SOD27_P7.62mm_Horizontal, F.Cu at (120.8, 118.8)
Connections:
- SW3 pad 2: Net-(D1-K) -> Net-(D5-A)
Routing:
- net Net-(D5-A): track 0.00 -> 84.8 mm
- net Net-(D1-K): track 84.7 -> 67.5 mm
- net Net-(D6-K): track 64.7 -> 72.4 mm

Commit message: Added BOM calculation
Other:
- board text added: "Clock board v1.0 P. Dovgalyuk, 2026"
- board text removed: "Clock board rev8 P. Dovgalyuk, 2026"
Changed lines of the file:
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@@
 		)
 	)
-	(gr_text "Clock board rev8\nP. Dovgalyuk, 2026"
+	(gr_text "Clock board v1.0\nP. Dovgalyuk, 2026"
 		(at 184 133.5 0)
 		(layer "B.SilkS")
