File: modules/decoder/decoder.kicad_pcb (KiCad board)
At the start: 2 copper layers, 108.2 x 140 mm, 27 parts, among them J10 Conn_02x05_Odd_Even, J13 Conn_02x04_Odd_Even, J16 Conn_01x04, K1 4PDT, K2 4PDT, K3 4PDT, K4 4PDT, K5 4PDT, K6 4PDT

Commit message: Added BOM calculation
Parts:
- D1, D2, D3, D4, D5, D6: footprint Diode_THT:D_DO-41_SOD81_P10.16mm_Horizontal -> Diode_THT:D_DO-35_SOD27_P7.62mm_Horizontal
- J13: footprint Connector_PinSocket_2.54mm:PinSocket_2x04_P2.54mm_Vertical -> Connector_PinHeader_2.54mm:PinHeader_2x04_P2.54mm_Vertical
- J16: footprint Connector_PinSocket_2.54mm:PinSocket_1x04_P2.54mm_Vertical -> Connector_PinHeader_2.54mm:PinHeader_1x04_P2.54mm_Vertical
- moved J13 2.48 mm to (95.7, 70.0)
Connections:
- J13 pad 1: Net-(J11-D0) -> Net-(J13-Pin_1)
- J13 pad 2: Net-(J13-Pin_2) -> Net-(J11-D0)
- J13 pad 3: Net-(J11-D1) -> Net-(J13-Pin_3)
- J13 pad 4: Net-(J13-Pin_4) -> Net-(J11-D1)
- J13 pad 5: Net-(J11-D2) -> Net-(J13-Pin_5)
- J13 pad 6: Net-(J13-Pin_6) -> Net-(J11-D2)
- J13 pad 7: Net-(J11-D3) -> Net-(J13-Pin_7)
- J13 pad 8: Net-(J13-Pin_8) -> Net-(J11-D3)
- K3 pad 10: Net-(J13-Pin_6) -> Net-(J13-Pin_5)
- K3 pad 11: Net-(J13-Pin_4) -> Net-(J13-Pin_3)
- K3 pad 12: Net-(J13-Pin_2) -> Net-(J13-Pin_1)
- K3 pad 9: Net-(J13-Pin_8) -> Net-(J13-Pin_7)
- K4 pad 10: Net-(J13-Pin_6) -> Net-(J13-Pin_5)
- K4 pad 11: Net-(J13-Pin_4) -> Net-(J13-Pin_3)
- K4 pad 12: Net-(J13-Pin_2) -> Net-(J13-Pin_1)
- K4 pad 9: Net-(J13-Pin_8) -> Net-(J13-Pin_7)
- K5 pad 10: Net-(J13-Pin_6) -> Net-(J13-Pin_5)
- K5 pad 11: Net-(J13-Pin_4) -> Net-(J13-Pin_3)
- K5 pad 12: Net-(J13-Pin_2) -> Net-(J13-Pin_1)
- K5 pad 9: Net-(J13-Pin_8) -> Net-(J13-Pin_7)
- K6 pad 10: Net-(J13-Pin_6) -> Net-(J13-Pin_5)
- K6 pad 11: Net-(J13-Pin_4) -> Net-(J13-Pin_3)
- K6 pad 12: Net-(J13-Pin_2) -> Net-(J13-Pin_1)
- K6 pad 9: Net-(J13-Pin_8) -> Net-(J13-Pin_7)
Routing:
- net Net-(J13-Pin_6): track 142.7 -> 0.00 mm
- net Net-(J13-Pin_8): track 142.6 -> 0.00 mm
- net Net-(J13-Pin_7): track 0.00 -> 142.5 mm
- net Net-(J13-Pin_5): track 0.00 -> 140.5 mm
- net Net-(J13-Pin_4): track 140.4 -> 0.00 mm
- net Net-(J13-Pin_3): track 0.00 -> 139.4 mm
- net Net-(J13-Pin_2): track 138.1 -> 0.00 mm
- net Net-(J13-Pin_1): track 0.00 -> 137.5 mm
- net Net-(J5-D3): track 19.4 -> 21.5 mm
- net Net-(J4-D3): track 19.4 -> 21.3 mm
- net Net-(J8-D3): track 19.4 -> 20.8 mm
- net Net-(J6-D3): track 19.4 -> 20.3 mm
Other:
- board text added: "Decoder board v1.0 P. Dovgalyuk, 2026"
- board text removed: "Decoder board rev6 P. Dovgalyuk, 2026"
