File: modules/matrix/matrix.kicad_pcb (KiCad board)
At the start: 2 copper layers, 57.8 x 57.8 mm, 18 parts, among them J10 Conn_C, J11 Conn_C, J12 Conn_D, J13 Conn_D, J14 Conn_Power2, J5 Conn_Power1, J6 Conn_A, J7 Conn_B, J8 Conn_B, J9 Conn_A

Commit message: Added BOM calculation
Other:
- board text added: "Matrix board v1.0 P. Dovgalyuk, 2026"
- board text removed: "Matrix board rev6 P. Dovgalyuk, 2026"
Changed lines of the file:
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@@
 		(property ki_fp_filters "Connector*:*_1x??_*")
 		(sheetname "/")
-		(sheetfile "switchboard.kicad_sch")
+		(sheetfile "matrix.kicad_sch")
 		(attr through_hole)
 		(fp_line
@@
 		(property ki_fp_filters "Connector*:*_1x??_*")
 		(sheetname "/")
-		(sheetfile "switchboard.kicad_sch")
+		(sheetfile "matrix.kicad_sch")
 		(attr through_hole)
 		(fp_line
@@
 		)
 		(sheetname "/")
-		(sheetfile "switchboard.kicad_sch")
+		(sheetfile "matrix.kicad_sch")
 		(attr through_hole)
 		(fp_line
@@
 		(property ki_fp_filters "Connector*:*_1x??_*")
 		(sheetname "/")
-		(sheetfile "switchboard.kicad_sch")
+		(sheetfile "matrix.kicad_sch")
 		(attr through_hole)
 		(fp_line
@@
 		(property ki_fp_filters "Connector*:*_1x??_*")
 		(sheetname "/")
-		(sheetfile "switchboard.kicad_sch")
+		(sheetfile "matrix.kicad_sch")
 		(attr through_hole)
 		(fp_line
@@
 		)
 		(sheetname "/")
-		(sheetfile "switchboard.kicad_sch")
+		(sheetfile "matrix.kicad_sch")
 		(attr through_hole)
 		(fp_line
@@
 		)
 		(sheetname "/")
-		(sheetfile "switchboard.kicad_sch")
+		(sheetfile "matrix.kicad_sch")
 		(attr through_hole)
 		(fp_line
@@
 		)
 		(sheetname "/")
-		(sheetfile "switchboard.kicad_sch")
+		(sheetfile "matrix.kicad_sch")
 		(attr through_hole)
 		(fp_line
@@
 		)
 		(sheetname "/")
-		(sheetfile "switchboard.kicad_sch")
+		(sheetfile "matrix.kicad_sch")
 		(attr through_hole)
 		(fp_line
@@
 		(property ki_fp_filters "Connector*:*_1x??_*")
 		(sheetname "/")
-		(sheetfile "switchboard.kicad_sch")
+		(sheetfile "matrix.kicad_sch")
 		(attr through_hole)
 		(fp_line
@@
 		(property ki_fp_filters "Connector*:*_1x??_*")
 		(sheetname "/")
-		(sheetfile "switchboard.kicad_sch")
+		(sheetfile "matrix.kicad_sch")
 		(attr through_hole)
 		(fp_line
@@
 		)
 		(sheetname "/")
-		(sheetfile "switchboard.kicad_sch")
+		(sheetfile "matrix.kicad_sch")
 		(attr through_hole)
 		(fp_line
@@
 		(property ki_fp_filters "Connector*:*_1x??_*")
 		(sheetname "/")
-		(sheetfile "switchboard.kicad_sch")
+		(sheetfile "matrix.kicad_sch")
 		(attr through_hole)
 		(fp_line
@@
 		)
 		(sheetname "/")
-		(sheetfile "switchboard.kicad_sch")
+		(sheetfile "matrix.kicad_sch")
 		(attr through_hole)
 		(fp_line
@@
 		(property ki_fp_filters "Connector*:*_1x??_*")
 		(sheetname "/")
-		(sheetfile "switchboard.kicad_sch")
+		(sheetfile "matrix.kicad_sch")
 		(attr through_hole)
 		(fp_line
@@
 		(property ki_fp_filters "Connector*:*_1x??_*")
 		(sheetname "/")
-		(sheetfile "switchboard.kicad_sch")
+		(sheetfile "matrix.kicad_sch")
 		(attr through_hole)
 		(fp_line
@@
 		)
 		(sheetname "/")
-		(sheetfile "switchboard.kicad_sch")
+		(sheetfile "matrix.kicad_sch")
 		(attr through_hole)
 		(fp_line
@@
 		(property ki_fp_filters "Connector*:*_1x??_*")
 		(sheetname "/")
-		(sheetfile "switchboard.kicad_sch")
+		(sheetfile "matrix.kicad_sch")
 		(attr through_hole)
 		(fp_line
@@
 		(layer "Edge.Cuts")
 	)
-	(gr_text "3"
-		(at 156.5 91.58 90)
+	(gr_text "0"
+		(at 139 98.77 0)
 		(layer "F.SilkS")
 		(effects
@@
 		)
 	)
-	(gr_text "0"
-		(at 148 91.58 90)
+	(gr_text "1"
+		(at 139 101.603333 0)
 		(layer "F.SilkS")
 		(effects
@@
 		)
 	)
-	(gr_text "0"
-		(at 147.75 113.75 90)
+	(gr_text "3"
+		(at 139 107.27 0)
 		(layer "F.SilkS")
 		(effects
@@
 		)
 	)
-	(gr_text "B"
-		(at 162 80.75 0)
+	(gr_text "+V"
+		(at 142.25 96 0)
 		(layer "F.SilkS")
 		(effects
 			(font
-				(size 4 4)
-				(thickness 0.5)
+				(size 2 2)
+				(thickness 0.25)
 			)
 			(justify left bottom)
 		)
 	)
-	(gr_text "D"
-		(at 149 111.25 0)
+	(gr_text "+V"
+		(at 154.5 110 0)
 		(layer "F.SilkS")
 		(effects
 			(font
-				(size 4 4)
-				(thickness 0.5)
+				(size 2 2)
+				(thickness 0.25)
 			)
 			(justify left bottom)
 		)
 	)
-	(gr_text "1"
-		(at 150.583333 113.75 90)
+	(gr_text "0"
+		(at 160.46 98.25 0)
 		(layer "F.SilkS")
 		(effects
@@
 		)
 	)
-	(gr_text "0"
-		(at 139 98.77 0)
+	(gr_text "1"
+		(at 160.46 101.083333 0)
 		(layer "F.SilkS")
 		(effects
@@
 		)
 	)
-	(gr_text "1"
-		(at 160.46 101.083333 0)
+	(gr_text "2"
+		(at 160.46 103.916667 0)
 		(layer "F.SilkS")
 		(effects
@@
 		)
 	)
-	(gr_text "A"
-		(at 125 89.75 0)
+	(gr_text "0"
+		(at 147.75 113.75 90)
 		(layer "F.SilkS")
 		(effects
 			(font
-				(size 4 4)
-				(thickness 0.5)
+				(size 2 2)
+				(thickness 0.25)
 			)
 			(justify left bottom)
 		)
 	)
-	(gr_text "+V"
-		(at 142.25 96 0)
+	(gr_text "0"
+		(at 148 91.58 90)
 		(layer "F.SilkS")
 		(effects
@@
 		)
 	)
-	(gr_text "Matrix"
-		(at 119 132.75 0)
+	(gr_text "1"
+		(at 150.583333 113.75 90)
 		(layer "F.SilkS")
 		(effects
 			(font
-				(size 4 4)
-				(thickness 0.5)
+				(size 2 2)
+				(thickness 0.25)
 			)
 			(justify left bottom)
@@
 		)
 	)
-	(gr_text "C"
-		(at 156 103.75 0)
+	(gr_text "2"
+		(at 153.416667 113.75 90)
 		(layer "F.SilkS")
 		(effects
 			(font
-				(size 4 4)
-				(thickness 0.5)
+				(size 2 2)
+				(thickness 0.25)
 			)
 			(justify left bottom)
 		)
 	)
-	(gr_text "3"
-		(at 139 107.27 0)
+	(gr_text "2"
+		(at 153.666667 91.58 90)
 		(layer "F.SilkS")
 		(effects
@@
 		)
 	)
-	(gr_text "C"
-		(at 172 117.5 0)
+	(gr_text "3"
+		(at 156.5 91.58 90)
 		(layer "F.SilkS")
 		(effects
 			(font
-				(size 4 4)
-				(thickness 0.5)
+				(size 2 2)
+				(thickness 0.25)
 			)
 			(justify left bottom)
 		)
 	)
-	(gr_text "A"
-		(at 141.5 104 0)
+	(gr_text "Matrix"
+		(at 119 132.75 0)
 		(layer "F.SilkS")
 		(effects
@@
 		)
 	)
-	(gr_text "+V"
-		(at 154.5 110 0)
+	(gr_text "A"
+		(at 125 89.75 0)
 		(layer "F.SilkS")
 		(effects
 			(font
-				(size 2 2)
-				(thickness 0.25)
+				(size 4 4)
+				(thickness 0.5)
 			)
 			(justify left bottom)
 		)
 	)
-	(gr_text "2"
-		(at 153.666667 91.58 90)
+	(gr_text "D"
+		(at 135.5 128 0)
 		(layer "F.SilkS")
 		(effects
 			(font
-				(size 2 2)
-				(thickness 0.25)
+				(size 4 4)
+				(thickness 0.5)
 			)
 			(justify left bottom)
 		)
 	)
-	(gr_text "1"
-		(at 139 101.603333 0)
+	(gr_text "A"
+		(at 141.5 104 0)
 		(layer "F.SilkS")
 		(effects
 			(font
-				(size 2 2)
-				(thickness 0.25)
+				(size 4 4)
+				(thickness 0.5)
 			)
 			(justify left bottom)
@@
 		)
 	)
-	(gr_text "0"
-		(at 160.46 98.25 0)
+	(gr_text "D"
+		(at 149 111.25 0)
 		(layer "F.SilkS")
 		(effects
 			(font
-				(size 2 2)
-				(thickness 0.25)
+				(size 4 4)
+				(thickness 0.5)
 			)
 			(justify left bottom)
 		)
 	)
-	(gr_text "D"
-		(at 135.5 128 0)
+	(gr_text "C"
+		(at 156 103.75 0)
 		(layer "F.SilkS")
 		(effects
@@
 		)
 	)
-	(gr_text "2"
-		(at 153.416667 113.75 90)
+	(gr_text "B"
+		(at 162 80.75 0)
 		(layer "F.SilkS")
 		(effects
 			(font
-				(size 2 2)
-				(thickness 0.25)
+				(size 4 4)
+				(thickness 0.5)
 			)
 			(justify left bottom)
 		)
 	)
-	(gr_text "2"
-		(at 160.46 103.916667 0)
+	(gr_text "C"
+		(at 172 117.5 0)
 		(layer "F.SilkS")
 		(effects
 			(font
-				(size 2 2)
-				(thickness 0.25)
+				(size 4 4)
+				(thickness 0.5)
 			)
 			(justify left bottom)
 		)
 	)
-	(gr_text "Matrix board rev6\nP. Dovgalyuk, 2026"
+	(gr_text "Matrix board v1.0\nP. Dovgalyuk, 2026"
 		(at 176.25 132.75 0)
 		(layer "B.SilkS")
