File: modules/register/register.kicad_pcb (KiCad board)
At the start: 2 copper layers, 113 x 103.5 mm, 30 parts, among them K0 4PDT, K1 4PDT, K2 4PDT, K3 4PDT

Commit message: Added BOM calculation
Other:
- board text added: "Register board v1.0 P. Dovgalyuk, 2026"
- board text removed: "Register board rev6 P. Dovgalyuk, 2026"
Changed lines of the file:
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@@
 		(layer "Edge.Cuts")
+	)
+	(gr_text "Control"
+		(at 89.5 60.5 0)
+		(layer "F.SilkS")
+		(effects
+			(font
+				(size 1 1)
+				(thickness 0.15)
+			)
+			(justify left bottom)
+		)
+	)
+	(gr_text "3"
+		(at 98.5 138.5 0)
+		(layer "F.SilkS")
+		(effects
+			(font
+				(size 4 4)
+				(thickness 0.15)
+			)
+			(justify left bottom)
+		)
+	)
+	(gr_text "2"
+		(at 123 138.5 0)
+		(layer "F.SilkS")
+		(effects
+			(font
+				(size 4 4)
+				(thickness 0.15)
+			)
+			(justify left bottom)
+		)
+	)
+	(gr_text "1"
+		(at 147.5 138.5 0)
+		(layer "F.SilkS")
+		(effects
+			(font
+				(size 4 4)
+				(thickness 0.15)
+			)
+			(justify left bottom)
+		)
 	)
 	(gr_text "0"
@@
 		)
 	)
-	(gr_text "Control"
-		(at 89.5 60.5 0)
-		(layer "F.SilkS")
-		(effects
-			(font
-				(size 1 1)
-				(thickness 0.15)
-			)
-			(justify left bottom)
-		)
-	)
-	(gr_text "2"
-		(at 123 138.5 0)
-		(layer "F.SilkS")
-		(effects
-			(font
-				(size 4 4)
-				(thickness 0.15)
-			)
-			(justify left bottom)
-		)
-	)
 	(gr_text "Register"
 		(at 88 55.5 0)
@@
 		)
 	)
-	(gr_text "1"
-		(at 147.5 138.5 0)
-		(layer "F.SilkS")
-		(effects
-			(font
-				(size 4 4)
-				(thickness 0.15)
-			)
-			(justify left bottom)
-		)
-	)
-	(gr_text "3"
-		(at 98.5 138.5 0)
-		(layer "F.SilkS")
-		(effects
-			(font
-				(size 4 4)
-				(thickness 0.15)
-			)
-			(justify left bottom)
-		)
-	)
-	(gr_text "Register board rev6\nP. Dovgalyuk, 2026"
+	(gr_text "Register board v1.0\nP. Dovgalyuk, 2026"
 		(at 199 149 0)
 		(layer "B.SilkS")
@@
 		)
 	)
+	(gr_text "Сброс"
+		(at 102.5 87.25 0)
+		(layer "Dwgs.User")
+		(effects
+			(font
+				(size 3 3)
+				(thickness 0.375)
+			)
+			(justify left bottom)
+		)
+	)
+	(gr_text "Реле-триггеры (хранение данных)"
+		(at 105.5 118.5 0)
+		(layer "Dwgs.User")
+		(effects
+			(font
+				(size 3 3)
+				(thickness 0.375)
+			)
+			(justify left bottom)
+		)
+	)
+	(gr_text "Шина 1"
+		(at 125 38 0)
+		(layer "Dwgs.User")
+		(effects
+			(font
+				(size 3 3)
+				(thickness 0.375)
+			)
+			(justify left bottom)
+		)
+	)
+	(gr_text "Шина 1"
+		(at 125.5 156 0)
+		(layer "Dwgs.User")
+		(effects
+			(font
+				(size 3 3)
+				(thickness 0.375)
+			)
+			(justify left bottom)
+		)
+	)
+	(gr_text "Шинные формирователи"
+		(at 129.75 87.25 0)
+		(layer "Dwgs.User")
+		(effects
+			(font
+				(size 3 3)
+				(thickness 0.375)
+			)
+			(justify left bottom)
+		)
+	)
+	(gr_text "Шина 2"
+		(at 149.5 38 0)
+		(layer "Dwgs.User")
+		(effects
+			(font
+				(size 3 3)
+				(thickness 0.375)
+			)
+			(justify left bottom)
+		)
+	)
+	(gr_text "Шина 2"
+		(at 149.5 156 0)
+		(layer "Dwgs.User")
+		(effects
+			(font
+				(size 3 3)
+				(thickness 0.375)
+			)
+			(justify left bottom)
+		)
+	)
+	(gr_text "Шина 3"
+		(at 174 38 0)
+		(layer "Dwgs.User")
+		(effects
+			(font
+				(size 3 3)
+				(thickness 0.375)
+			)
+			(justify left bottom)
+		)
+	)
+	(gr_text "Шина 3"
+		(at 174 156 0)
+		(layer "Dwgs.User")
+		(effects
+			(font
+				(size 3 3)
+				(thickness 0.375)
+			)
+			(justify left bottom)
+		)
+	)
 	(gr_text "Управляющие сигналы"
 		(at 82.75 97.75 90)
@@
 		)
 	)
-	(gr_text "Шина 3"
-		(at 174 38 0)
-		(layer "Dwgs.User")
-		(effects
-			(font
-				(size 3 3)
-				(thickness 0.375)
-			)
-			(justify left bottom)
-		)
-	)
-	(gr_text "Шина 3"
-		(at 174 156 0)
+	(gr_text "Биты 0-3"
+		(at 83 126.5 90)
+		(layer "Dwgs.User")
+		(effects
+			(font
+				(size 3 3)
+				(thickness 0.375)
+			)
+			(justify left bottom)
+		)
+	)
+	(gr_text "Биты 2-3"
+		(at 83 153 90)
 		(layer "Dwgs.User")
 		(effects
@@
 		)
 	)
-	(gr_text "Шина 2"
-		(at 149.5 38 0)
-		(layer "Dwgs.User")
-		(effects
-			(font
-				(size 3 3)
-				(thickness 0.375)
-			)
-			(justify left bottom)
-		)
-	)
-	(gr_text "Биты 2-3"
-		(at 83 153 90)
-		(layer "Dwgs.User")
-		(effects
-			(font
-				(size 3 3)
-				(thickness 0.375)
-			)
-			(justify left bottom)
-		)
-	)
 	(gr_text "Управляющие реле"
 		(at 108.75 81.25 0)
@@
 			)
 			(justify left bottom)
-		)
-	)
-	(gr_text "Шина 2"
-		(at 149.5 156 0)
-		(layer "Dwgs.User")
-		(effects
-			(font
-				(size 3 3)
-				(thickness 0.375)
-			)
-			(justify left bottom)
-		)
-	)
-	(gr_text "Шина 1"
-		(at 125 38 0)
-		(layer "Dwgs.User")
-		(effects
-			(font
-				(size 3 3)
-				(thickness 0.375)
-			)
-			(justify left bottom)
-		)
-	)
-	(gr_text "Шинные формирователи"
-		(at 129.75 87.25 0)
-		(layer "Dwgs.User")
-		(effects
-			(font
-				(size 3 3)
-				(thickness 0.375)
-			)
-			(justify left bottom)
-		)
-	)
-	(gr_text "Реле-триггеры (хранение данных)"
-		(at 105.5 118.5 0)
-		(layer "Dwgs.User")
-		(effects
-			(font
-				(size 3 3)
-				(thickness 0.375)
-			)
-			(justify left bottom)
-		)
-	)
-	(gr_text "Биты 0-3"
-		(at 83 126.5 90)
-		(layer "Dwgs.User")
-		(effects
-			(font
-				(size 3 3)
-				(thickness 0.375)
-			)
-			(justify left bottom)
-		)
-	)
-	(gr_text "Шина 1"
-		(at 125.5 156 0)
-		(layer "Dwgs.User")
-		(effects
-			(font
-				(size 3 3)
-				(thickness 0.375)
-			)
-			(justify left bottom)
-		)
-	)
-	(gr_text "Сброс"
-		(at 102.5 87.25 0)
-		(layer "Dwgs.User")
-		(effects
-			(font
-				(size 3 3)
-				(thickness 0.375)
-			)
-			(justify left bottom)
