File: modules/rom/rom.kicad_pcb (KiCad board)
At the start: 2 copper layers, 126.8 x 77 mm, 65 parts, among them J14 Conn_02x05_Odd_Even, K1 4PDT, K2 4PDT, SW1 SW_DIP_x04, SW2 SW_DIP_x04, SW3 SW_DIP_x04, SW4 SW_DIP_x04, SW5 SW_DIP_x04, SW6 SW_DIP_x04, SW7 SW_DIP_x04, SW8 SW_DIP_x04

Commit message: Updated actions
Parts:
- moved D1 52.6 mm to (137.1, 66.8)
- moved D2 52.6 mm to (137.1, 78.3)
- moved D3 52.6 mm to (137.1, 89.8)
- moved D4 52.6 mm to (137.1, 101.3)
- moved D12 52.6 mm to (164.0, 68.3)
- moved D13 52.6 mm to (167.4, 71.2)
- moved D14 52.6 mm to (166.2, 74.0)
- moved D16 52.6 mm to (164.0, 79.8)
- moved D18 52.6 mm to (166.2, 85.5)
- moved D20 52.6 mm to (164.0, 91.3)
- moved D21 52.6 mm to (167.4, 94.1)
- moved D22 52.6 mm to (166.2, 97.0)
- moved D23 52.6 mm to (165.2, 99.9)
- moved D24 52.6 mm to (164.0, 102.7)
- moved D28 52.6 mm to (191.4, 68.4)
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Other:
- board text added: "Сигнал выборки"
- board text added: "Шина адреса"
- board text added: "Шина данных"

Commit message: Added BOM calculation
Parts:
- D41, D42: footprint Diode_THT:D_DO-41_SOD81_P10.16mm_Horizontal -> Diode_THT:D_DO-35_SOD27_P7.62mm_Horizontal
- moved D42 1.51 mm to (109.5, 87.8)
- moved D41 1.27 mm to (109.2, 125.3)
Routing:
- net Net-(D42-K): track 151.6 -> 152.9 mm
Other:
- board text added: "ROM board v1.0 P. Dovgalyuk, 2026"
- board text removed: "ROM board rev7 P. Dovgalyuk, 2026"
Changed lines of the file:
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@@
 		)
 	)
-	(footprint "Diode_THT:D_DO-41_SOD81_P10.16mm_Horizontal"
+	(footprint "Diode_THT:D_DO-35_SOD27_P7.62mm_Horizontal"
 		(layer "F.Cu")
-		(at 107.97 125.311492)
-		(descr "Diode, DO-41_SOD81 series, Axial, Horizontal, pin pitch=10.16mm, length*diameter=5.2*2.7mm^2, https://www.diodes.com/assets/Package-Files/DO-41-Plastic.pdf")
-		(tags "Diode DO-41_SOD81 series Axial Horizontal pin pitch 10.16mm  length 5.2mm diameter 2.7mm")
+		(at 109.24 125.27)
+		(descr "Diode, DO-35_SOD27 series, Axial, Horizontal, pin pitch=7.62mm, length*diameter=4*2mm^2, http://www.diodes.com/_files/packages/DO-35.pdf")
+		(tags "Diode DO-35_SOD27 series Axial Horizontal pin pitch 7.62mm  length 4mm diameter 2mm")
 		(property "Reference" "D41"
-			(at 5.08 -2.47 0)
+			(at 3.81 -2.12 0)
 			(layer "F.SilkS")
 			(hide yes)
@@
 		)
 		(property "Value" "1N4001"
-			(at 5.08 2.47 0)
+			(at 3.81 2.12 0)
 			(layer "F.Fab")
 			(hide yes)
@@
 		(attr through_hole)
 		(fp_line
-			(start 1.34 0)
-			(end 2.36 0)
+			(start 1.04 0)
+			(end 1.69 0)
 			(stroke
 				(width 0.12)
@@
 		)
 		(fp_line
-			(start 3.14 -1.47)
-			(end 3.14 1.47)
+			(start 2.29 -1.12)
+			(end 2.29 1.12)
 			(stroke
 				(width 0.12)
@@
 		)
 		(fp_line
-			(start 3.26 -1.47)
-			(end 3.26 1.47)
+			(start 2.41 -1.12)
+			(end 2.41 1.12)
 			(stroke
 				(width 0.12)
@@
 		)
 		(fp_line
-			(start 3.38 -1.47)
-			(end 3.38 1.47)
+			(start 2.53 -1.12)
+			(end 2.53 1.12)
 			(stroke
 				(width 0.12)
@@
 		)
 		(fp_line
-			(start 8.82 0)
-			(end 7.8 0)
+			(start 6.58 0)
+			(end 5.93 0)
 			(stroke
 				(width 0.12)
@@
 		)
 		(fp_rect
-			(start 2.36 -1.47)
-			(end 7.8 1.47)
+			(start 1.69 -1.12)
+			(end 5.93 1.12)
 			(stroke
 				(width 0.12)
@@
 		)
 		(fp_rect
-			(start -1.35 -1.6)
-			(end 11.51 1.6)
+			(start -1.05 -1.25)
+			(end 8.67 1.25)
 			(stroke
 				(width 0.05)
@@
 		(fp_line
 			(start 0 0)
-			(end 2.48 0)
+			(end 1.81 0)
 			(stroke
 				(width 0.1)
@@
 		)
 		(fp_line
-			(start 3.16 -1.35)
-			(end 3.16 1.35)
+			(start 2.31 -1)
+			(end 2.31 1)
 			(stroke
 				(width 0.1)
@@
 		)
 		(fp_line
-			(start 3.26 -1.35)
-			(end 3.26 1.35)
+			(start 2.41 -1)
+			(end 2.41 1)
 			(stroke
 				(width 0.1)
@@
 		)
 		(fp_line
-			(start 3.36 -1.35)
-			(end 3.36 1.35)
+			(start 2.51 -1)
+			(end 2.51 1)
 			(stroke
 				(width 0.1)
@@
 		)
 		(fp_line
-			(start 10.16 0)
-			(end 7.68 0)
+			(start 7.62 0)
+			(end 5.81 0)
 			(stroke
 				(width 0.1)
@@
 		)
 		(fp_rect
-			(start 2.48 -1.35)
-			(end 7.68 1.35)
+			(start 1.81 -1)
+			(end 5.81 1)
 			(stroke
 				(width 0.1)
@@
 		(pad "1" thru_hole roundrect
 			(at 0 0)
-			(size 2.2 2.2)
-			(drill 1.1)
+			(size 1.6 1.6)
+			(drill 0.8)
 			(layers "*.Cu" "*.Mask")
 			(remove_unused_layers no)
-			(roundrect_rratio 0.113636)
+			(roundrect_rratio 0.15625)
 			(net 1 "Net-(D41-K)")
 			(pinfunction "K")
@@
 		)
 		(pad "2" thru_hole circle
-			(at 10.16 0)
-			(size 2.2 2.2)
-			(drill 1.1)
+			(at 7.62 0)
+			(size 1.6 1.6)
+			(drill 0.8)
 			(layers "*.Cu" "*.Mask")
 			(remove_unused_layers no)
@@
 		)
 		(embedded_fonts no)
-		(model "${KICAD9_3DMODEL_DIR}/Diode_THT.3dshapes/D_DO-41_SOD81_P10.16mm_Horizontal.step"
+		(model "${KICAD9_3DMODEL_DIR}/Diode_THT.3dshapes/D_DO-35_SOD27_P7.62mm_Horizontal.step"
 			(offset
 				(xyz 0 0 0)
@@
 		)
 	)
-	(footprint "Diode_THT:D_DO-41_SOD81_P10.16mm_Horizontal"
+	(footprint "Diode_THT:D_DO-35_SOD27_P7.62mm_Horizontal"
 		(layer "F.Cu")
-		(at 107.97 87.811492)
-		(descr "Diode, DO-41_SOD81 series, Axial, Horizontal, pin pitch=10.16mm, length*diameter=5.2*2.7mm^2, https://www.diodes.com/assets/Package-Files/DO-41-Plastic.pdf")
-		(tags "Diode DO-41_SOD81 series Axial Horizontal pin pitch 10.16mm  length 5.2mm diameter 2.7mm")
+		(at 109.48 87.82)
+		(descr "Diode, DO-35_SOD27 series, Axial, Horizontal, pin pitch=7.62mm, length*diameter=4*2mm^2, http://www.diodes.com/_files/packages/DO-35.pdf")
+		(tags "Diode DO-35_SOD27 series Axial Horizontal pin pitch 7.62mm  length 4mm diameter 2mm")
 		(property "Reference" "D42"
-			(at 5.08 -2.47 0)
+			(at 3.81 -2.12 0)
 			(layer "F.SilkS")
 			(hide yes)
@@
 		)
 		(property "Value" "1N4001"
-			(at 5.08 2.47 0)
+			(at 3.81 2.12 0)
 			(layer "F.Fab")
 			(hide yes)
@@
 		(attr through_hole)
 		(fp_line
-			(start 1.34 0)
-			(end 2.36 0)
+			(start 1.04 0)
+			(end 1.69 0)
 			(stroke
 				(width 0.12)
@@
 		)
 		(fp_line
-			(start 3.14 -1.47)
-			(end 3.14 1.47)
+			(start 2.29 -1.12)
+			(end 2.29 1.12)
 			(stroke
 				(width 0.12)
@@
 		)
 		(fp_line
-			(start 3.26 -1.47)
-			(end 3.26 1.47)
+			(start 2.41 -1.12)
+			(end 2.41 1.12)
 			(stroke
 				(width 0.12)
@@
 		)
 		(fp_line
-			(start 3.38 -1.47)
-			(end 3.38 1.47)
+			(start 2.53 -1.12)
+			(end 2.53 1.12)
 			(stroke
 				(width 0.12)
@@
 		)
 		(fp_line
-			(start 8.82 0)
-			(end 7.8 0)
+			(start 6.58 0)
+			(end 5.93 0)
 			(stroke
 				(width 0.12)
@@
 		)
 		(fp_rect
-			(start 2.36 -1.47)
-			(end 7.8 1.47)
+			(start 1.69 -1.12)
+			(end 5.93 1.12)
 			(stroke
 				(width 0.12)
@@
 		)
 		(fp_rect
-			(start -1.35 -1.6)
-			(end 11.51 1.6)
+			(start -1.05 -1.25)
+			(end 8.67 1.25)
 			(stroke
 				(width 0.05)
@@
 		(fp_line
 			(start 0 0)
-			(end 2.48 0)
+			(end 1.81 0)
 			(stroke
 				(width 0.1)
@@
 		)
 		(fp_line
-			(start 3.16 -1.35)
-			(end 3.16 1.35)
+			(start 2.31 -1)
+			(end 2.31 1)
 			(stroke
 				(width 0.1)
@@
 		)
 		(fp_line
-			(start 3.26 -1.35)
-			(end 3.26 1.35)
+			(start 2.41 -1)
+			(end 2.41 1)
 			(stroke
 				(width 0.1)
@@
 		)
 		(fp_line
-			(start 3.36 -1.35)
-			(end 3.36 1.35)
+			(start 2.51 -1)
+			(end 2.51 1)
 			(stroke
 				(width 0.1)
@@
 		)
 		(fp_line
-			(start 10.16 0)
-			(end 7.68 0)
+			(start 7.62 0)
+			(end 5.81 0)
 			(stroke
 				(width 0.1)
@@
 		)
 		(fp_rect
-			(start 2.48 -1.35)
-			(end 7.68 1.35)
+			(start 1.81 -1)
+			(end 5.81 1)
 			(stroke
 				(width 0.1)
@@
 		(pad "1" thru_hole roundrect
 			(at 0 0)
-			(size 2.2 2.2)
-			(drill 1.1)
+			(size 1.6 1.6)
+			(drill 0.8)
 			(layers "*.Cu" "*.Mask")
 			(remove_unused_layers no)
-			(roundrect_rratio 0.113636)
+			(roundrect_rratio 0.15625)
 			(net 2 "Net-(D42-K)")
 			(pinfunction "K")
@@
 		)
 		(pad "2" thru_hole circle
-			(at 10.16 0)
-			(size 2.2 2.2)
-			(drill 1.1)
+			(at 7.62 0)
+			(size 1.6 1.6)
+			(drill 0.8)
 			(layers "*.Cu" "*.Mask")
 			(remove_unused_layers no)
@@
 		)
 		(embedded_fonts no)
-		(model "${KICAD9_3DMODEL_DIR}/Diode_THT.3dshapes/D_DO-41_SOD81_P10.16mm_Horizontal.step"
+		(model "${KICAD9_3DMODEL_DIR}/Diode_THT.3dshapes/D_DO-35_SOD27_P7.62mm_Horizontal.step"
 			(offset
 				(xyz 0 0 0)
@@
 		)
 	)
-	(gr_text "ROM board rev7\nP. Dovgalyuk, 2026"
+	(gr_text "ROM board v1.0\nP. Dovgalyuk, 2026"
 		(at 201.65 127.811492 0)
 		(layer "B.SilkS")
@@
 	)
 	(segment
-		(start 107.97 125.311492)
-		(end 107.97 116.831492)
-		(width 0.2)
-		(layer "F.Cu")
-		(net 1)
-	)
-	(segment
 		(start 100.934281 109.795773)
 		(end 94.25 109.795773)
@@
 	)
 	(segment
+		(start 109.24 125.27)
+		(end 107.97 124)
+		(width 0.2)
+		(layer "F.Cu")
+		(net 1)
+	)
+	(segment
+		(start 107.97 124)
+		(end 107.97 116.831492)
+		(width 0.2)
+		(layer "F.Cu")
+		(net 1)
+	)
+	(segment
 		(start 106.45 115.311492)
 		(end 100.934281 109.795773)
@@
 	)
 	(segment
-		(start 107.97 87.811492)
+		(start 109.48 87.82)
+		(end 107.97 86.31)
+		(width 0.2)
+		(layer "F.Cu")
+		(net 2)
+	)
+	(segment
+		(start 107.97 86.31)
 		(end 107.97 79.381492)
 		(width 0.2)
@@
 	)
 	(segment
-		(start 107.97 93.295773)
-		(end 95.4 105.865773)
+		(start 109.48 87.82)
+		(end 107.97 89.33)
 		(width 0.2)
 		(layer "B.Cu")
@@
 	)
 	(segment
+		(start 107.97 93.295773)
+		(end 95.4 105.865773)
+		(width 0.2)
+		(layer "B.Cu")
+		(net 2)
+	)
+	(segment
 		(start 94.01 107.255773)
 		(end 95.4 105.865773)
@@
 	)
 	(segment
-		(start 89.53015 107.255773)
-		(end 94.01 107.255773)
+		(start 107.97 89.33)
+		(end 107.97 93.295773)
 		(width 0.2)
 		(layer "B.Cu")
@@
 	)
 	(segment
-		(start 200.15 103.325773)
-		(end 198.164281 105.311492)
+		(start 89.53015 107.255773)
+		(end 94.01 107.255773)
 		(width 0.2)
 		(layer "B.Cu")
@@
 	)
 	(segment
-		(start 107.97 87.811492)
-		(end 107.97 93.295773)
+		(start 200.15 103.325773)
+		(end 198.164281 105.311492)
 		(width 0.2)
 		(layer "B.Cu")
