File: modules/switches/switches.kicad_pcb (KiCad board)
At the start: 2 copper layers, 42.5 x 52 mm, 7 parts, among them SW1 SW_SPDT, SW2 SW_SPDT, SW3 SW_SPDT, SW4 SW_SPDT

Commit message: Added BOM calculation
Other:
- board text added: "Switches board v1.0 P. Dovgalyuk, 2026"
- board text removed: "Switches board rev6 P. Dovgalyuk, 2026"
Changed lines of the file:
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@@
 		(layer "Edge.Cuts")
 	)
-	(gr_text "D3"
-		(at 119.5 79.5 0)
+	(gr_text "BUS3"
+		(at 118.5 97.5 0)
 		(layer "F.SilkS")
 		(effects
 			(font
-				(size 3 3)
+				(size 2 2)
 				(thickness 0.1)
 			)
@@
 	(gr_text "BUS2"
 		(at 129 97.5 0)
+		(layer "F.SilkS")
+		(effects
+			(font
+				(size 2 2)
+				(thickness 0.1)
+			)
+			(justify left bottom)
+		)
+	)
+	(gr_text "BUS1"
+		(at 139.5 97.5 0)
 		(layer "F.SilkS")
 		(effects
@@
 		)
 	)
+	(gr_text "D3"
+		(at 119.5 79.5 0)
+		(layer "F.SilkS")
+		(effects
+			(font
+				(size 3 3)
+				(thickness 0.1)
+			)
+			(justify left bottom)
+		)
+	)
 	(gr_text "D2"
 		(at 130 79.5 0)
+		(layer "F.SilkS")
+		(effects
+			(font
+				(size 3 3)
+				(thickness 0.1)
+			)
+			(justify left bottom)
+		)
+	)
+	(gr_text "D1"
+		(at 140.5 79.5 0)
 		(layer "F.SilkS")
 		(effects
@@
 		)
 	)
-	(gr_text "BUS3"
-		(at 118.5 97.5 0)
+	(gr_text "0"
+		(at 120 104.5 0)
 		(layer "F.SilkS")
 		(effects
 			(font
-				(size 2 2)
+				(size 5 5)
 				(thickness 0.1)
 			)
@@
 		)
 	)
-	(gr_text "BUS1"
-		(at 139.5 97.5 0)
-		(layer "F.SilkS")
-		(effects
-			(font
-				(size 2 2)
-				(thickness 0.1)
-			)
-			(justify left bottom)
-		)
-	)
-	(gr_text "D1"
-		(at 140.5 79.5 0)
-		(layer "F.SilkS")
-		(effects
-			(font
-				(size 3 3)
-				(thickness 0.1)
-			)
-			(justify left bottom)
-		)
-	)
-	(gr_text "0"
-		(at 120 104.5 0)
+	(gr_text "1"
+		(at 151.5 75 0)
 		(layer "F.SilkS")
 		(effects
@@
 		)
 	)
-	(gr_text "1"
-		(at 151.5 75 0)
-		(layer "F.SilkS")
-		(effects
-			(font
-				(size 5 5)
-				(thickness 0.1)
-			)
-			(justify left bottom)
-		)
-	)
-	(gr_text "Switches board rev6\nP. Dovgalyuk, 2026"
+	(gr_text "Switches board v1.0\nP. Dovgalyuk, 2026"
 		(at 158.5 120 0)
 		(layer "B.SilkS")
