File: modules/unary/unary.kicad_pcb (KiCad board)
At the start: 2 copper layers, 121.5 x 85.5 mm, 19 parts, among them J10 COPY2, J11 COPY3, J3 IN, J4 IN, J5 NOT, J6 SHR, J7 NOT, J8 SHR, J9 COPY1, K1 4PDT, K2 4PDT, K3 4PDT, K4 4PDT

Commit message: Added BOM calculation
Other:
- board text added: "Unary logic board v1.0 P. Dovgalyuk, 2026"
- board text removed: "Unary logic board rev6 P. Dovgalyuk, 2026"
Changed lines of the file:
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@@
 			(drillshape 0)
 			(scaleselection 1)
-			(outputdirectory "../../gerber/rev4/logic_unary")
+			(outputdirectory "../../gerber/rev4/unary")
 		)
 	)
@@
 		)
 		(sheetname "/")
-		(sheetfile "logic_unary.kicad_sch")
+		(sheetfile "unary.kicad_sch")
 		(attr through_hole)
 		(fp_line
@@
 		)
 		(sheetname "/")
-		(sheetfile "logic_unary.kicad_sch")
+		(sheetfile "unary.kicad_sch")
 		(attr through_hole)
 		(fp_rect
@@
 		)
 		(sheetname "/")
-		(sheetfile "logic_unary.kicad_sch")
+		(sheetfile "unary.kicad_sch")
 		(attr through_hole)
 		(fp_rect
@@
 		(property ki_fp_filters "D*DO?35*")
 		(sheetname "/")
-		(sheetfile "logic_unary.kicad_sch")
+		(sheetfile "unary.kicad_sch")
 		(attr through_hole)
 		(fp_line
@@
 		(property ki_fp_filters "D*DO?35*")
 		(sheetname "/")
-		(sheetfile "logic_unary.kicad_sch")
+		(sheetfile "unary.kicad_sch")
 		(attr through_hole)
 		(fp_line
@@
 		)
 		(sheetname "/")
-		(sheetfile "logic_unary.kicad_sch")
+		(sheetfile "unary.kicad_sch")
 		(attr through_hole)
 		(fp_line
@@
 		)
 		(sheetname "/")
-		(sheetfile "logic_unary.kicad_sch")
+		(sheetfile "unary.kicad_sch")
 		(attr through_hole)
 		(fp_line
@@
 		)
 		(sheetname "/")
-		(sheetfile "logic_unary.kicad_sch")
+		(sheetfile "unary.kicad_sch")
 		(attr through_hole)
 		(fp_line
@@
 		)
 		(sheetname "/")
-		(sheetfile "logic_unary.kicad_sch")
+		(sheetfile "unary.kicad_sch")
 		(attr through_hole)
 		(fp_line
@@
 		)
 		(sheetname "/")
-		(sheetfile "logic_unary.kicad_sch")
+		(sheetfile "unary.kicad_sch")
 		(attr through_hole)
 		(fp_rect
@@
 		(property ki_fp_filters "D*DO?35*")
 		(sheetname "/")
-		(sheetfile "logic_unary.kicad_sch")
+		(sheetfile "unary.kicad_sch")
 		(attr through_hole)
 		(fp_line
@@
 		)
 		(sheetname "/")
-		(sheetfile "logic_unary.kicad_sch")
+		(sheetfile "unary.kicad_sch")
 		(attr through_hole)
 		(fp_rect
@@
 		)
 		(sheetname "/")
-		(sheetfile "logic_unary.kicad_sch")
+		(sheetfile "unary.kicad_sch")
 		(attr through_hole)
 		(fp_line
@@
 		)
 		(sheetname "/")
-		(sheetfile "logic_unary.kicad_sch")
+		(sheetfile "unary.kicad_sch")
 		(attr through_hole)
 		(fp_line
@@
 		)
 		(sheetname "/")
-		(sheetfile "logic_unary.kicad_sch")
+		(sheetfile "unary.kicad_sch")
 		(attr through_hole)
 		(fp_line
@@
 		)
 		(sheetname "/")
-		(sheetfile "logic_unary.kicad_sch")
+		(sheetfile "unary.kicad_sch")
 		(attr through_hole)
 		(fp_line
@@
 		)
 		(sheetname "/")
-		(sheetfile "logic_unary.kicad_sch")
+		(sheetfile "unary.kicad_sch")
 		(attr through_hole)
 		(fp_line
@@
 		)
 		(sheetname "/")
-		(sheetfile "logic_unary.kicad_sch")
+		(sheetfile "unary.kicad_sch")
 		(attr through_hole)
 		(fp_line
@@
 		(property ki_fp_filters "D*DO?35*")
 		(sheetname "/")
-		(sheetfile "logic_unary.kicad_sch")
+		(sheetfile "unary.kicad_sch")
 		(attr through_hole)
 		(fp_line
@@
 		(layer "Edge.Cuts")
 	)
-	(gr_text "NOT"
-		(at 147 95 0)
-		(layer "F.SilkS")
-		(effects
-			(font
-				(size 5 5)
-				(thickness 0.625)
-			)
-			(justify left bottom)
-		)
-	)
 	(gr_text "COPY"
 		(at 97.5 113.5 0)
@@
 		)
 	)
-	(gr_text "Unary"
-		(at 90 43.5 0)
+	(gr_text "NOT"
+		(at 147 95 0)
 		(layer "F.SilkS")
 		(effects
 			(font
-				(size 8 8)
-				(thickness 1)
+				(size 5 5)
+				(thickness 0.625)
 			)
 			(justify left bottom)
@@
 		)
 	)
-	(gr_text "Unary logic board rev6\nP. Dovgalyuk, 2026"
-		(at 210.5 39 0)
+	(gr_text "Unary"
+		(at 90 43.5 0)
+		(layer "F.SilkS")
+		(effects
+			(font
+				(size 8 8)
+				(thickness 1)
+			)
+			(justify left bottom)
+		)
+	)
+	(gr_text "Unary logic board v1.0\nP. Dovgalyuk, 2026"
+		(at 210.09 116.83 0)
 		(layer "B.SilkS")
 		(effects
@@
 		)
 	)
-	(gr_text "Входящий бит\nдля сдвига"
-		(at 86.5 73 90)
+	(gr_text "Операнд"
+		(at 131 23 0)
 		(layer "Dwgs.User")
 		(effects
@@
 		)
 	)
-	(gr_text "Копии операнда"
-		(at 87.5 115 90)
+	(gr_text "Результат сдвига"
+		(at 168.5 124.5 0)
 		(layer "Dwgs.User")
 		(effects
@@
 		)
 	)
-	(gr_text "Результат сдвига"
-		(at 168.5 124.5 0)
+	(gr_text "Входящий бит\nдля сдвига"
+		(at 86.5 73 90)
 		(layer "Dwgs.User")
 		(effects
@@
 		)
 	)
-	(gr_text "Выходной бит сдвига"
-		(at 226 90.5 90)
+	(gr_text "Копии операнда"
+		(at 87.5 115 90)
 		(layer "Dwgs.User")
 		(effects
@@
 		)
 	)
-	(gr_text "Операнд"
-		(at 131 23 0)
+	(gr_text "Выходной бит сдвига"
+		(at 226 90.5 90)
 		(layer "Dwgs.User")
 		(effects
